Commit message: Add catkin workspace

File: catkin_ws/src/robot_description/urdf/robotic-arm-3dof.urdf (robot description, URDF)
Before this commit: robot robotic-arm-3dof, 4 links, 3 joints
Links:
- link Cylinder.001_link: geometry collision box size=2.66965 0.80000 0.20000; visual mesh filename=package://robot_description/meshes/Cylinder.001.dae scale=1.00000 1.00000 1.00000
- link Cylinder.002_link: geometry collision box size=1.22719 0.40000 0.40000; visual mesh filename=package://robot_description/meshes/Cylinder.003.dae scale=1.00000 1.00000 1.00000
- link Cylinder.003_link: geometry collision box size=0.30000 0.30000 1.02500; visual mesh filename=package://robot_description/meshes/Cylinder.004.dae scale=1.00000 1.00000 1.00000
- link Cylinder_link: geometry visual mesh filename=package://robot_description/meshes/Cylinder.dae scale=1.00000 1.00000 1.00000

Commit message: Add fixed joint to world

File: catkin_ws/src/robot_description/urdf/robotic-arm-3dof.urdf (robot description, URDF)
Before this commit: robot robotic-arm-3dof, 4 links, 3 joints
Links:
- added link world
Joints:
- added joint fixed_to_world: type fixed, parent world, child Cylinder_link

Commit message: Update physics

File: catkin_ws/src/robot_description/urdf/robotic-arm-3dof.urdf (robot description, URDF)
Before this commit: robot robotic-arm-3dof, 5 links, 4 joints
Links:
- link Cylinder_link: mass 0.00001 -> 50

Commit message: Update URDF physics

File: catkin_ws/src/robot_description/urdf/robotic-arm-3dof.urdf (robot description, URDF)
Before this commit: robot robotic-arm-3dof, 5 links, 4 joints
Joints:
- joint joint_1: limit lower=-3.14000 upper=3.14000 effort=0.00000 velocity=0.00000 -> lower=-3.14000 upper=3.14000 effort=1e4 velocity=10
- joint joint_2: limit lower=-3.14000 upper=3.14000 effort=0.00000 velocity=0.00000 -> lower=-3.14000 upper=3.14000 effort=1e4 velocity=10
- joint joint_3: limit lower=-3.14000 upper=3.14000 effort=0.00000 velocity=0.00000 -> lower=-3.14000 upper=3.14000 effort=1e4 velocity=10
